Commit message: added sonar sensors to urdf

File: ros2_automower_description/description/robot_core.xacro (robot description, xacro)
@@ -109,3 +109,252 @@
         </xacro:inertial_sphere>
     </link>
+    <!-- SENSORS -->
+    <!-- SONAR SENSOR FRONT RIGHT -->
+    <joint name="sonar_front_right_joint" type="fixed">
+    <axis xyz="0 1 0" />
+    <origin rpy="0 0 0" xyz="0.41966 -0.039825 0.10134" />
+    <parent link="base_link"/>
+    <child link="base_sonar_front_right"/>
+    </joint>
+    <link name="base_sonar_front_right">
+        <collision>
+        <origin xyz="0 0 0" rpy="0 0 0"/>
+        <geometry>
+            <box size="0.01 0.01 0.01"/>
+        </geometry>
+        </collision>
+        <visual>
+        <origin xyz="0 0 0" rpy="0 0 0"/>
+        <geometry>
+            <box size="0.01 0.01 0.01"/>
+        </geometry>
+        </visual>
+        <inertial>
+        <mass value="1e-5" />
+        <origin xyz="0 0 0" rpy="0 0 0"/>
+        <inertia ixx="1e-6" ixy="0" ixz="0" iyy="1e-6" iyz="0" izz="1e-6" />
+        </inertial>
+    </link>
+    <gazebo reference="base_sonar_front_right">
+    <sensor type="ray" name="TeraRanger">
+        <pose>0 0 0 0 0 0</pose>
+        <visualize>true</visualize>
+        <update_rate>50</update_rate>
+        <ray>
+            <scan>
+                <horizontal>
+                <samples>10</samples>
+                <resolution>1</resolution>
+                <min_angle>-0.14835</min_angle>
+                <max_angle>0.14835</max_angle>
+                </horizontal>
+                <vertical>
+                <samples>10</samples>
+                <resolution>1</resolution>
+                <min_angle>-0.14835</min_angle>
+                <max_angle>0.14835</max_angle>
+                </vertical>
+            </scan>
+            <range>
+                <min>0.01</min>
+                <max>2</max>
+                <resolution>0.02</resolution>
+            </range>
+        </ray>
+        <plugin filename="libgazebo_ros_range.so" name="gazebo_ros_range">
+            <gaussianNoise>0.005</gaussianNoise>
+            <alwaysOn>true</alwaysOn>
+            <updateRate>50</updateRate>
+            <topicName>sensor/sonar_front_right</topicName>
+            <frameName>base_sonar_front_right</frameName>
+            <fov>0.2967</fov>
+        </plugin>
+    </sensor>
+    </gazebo>
+    <!-- SONAR SENSOR FRONT RIGHT -->
+    <joint name="sonar_front_left_joint" type="fixed">
+    <axis xyz="0 1 0" />
+    <origin rpy="0 0 0" xyz="0.41966 0.039825 0.10134" />
+    <parent link="base_link"/>
+    <child link="base_sonar_front_left"/>
+    </joint>
+    <link name="base_sonar_front_left">
+        <collision>
+        <origin xyz="0 0 0" rpy="0 0 0"/>
+        <geometry>
+            <box size="0.01 0.01 0.01"/>
+        </geometry>
+        </collision>
+        <visual>
+        <origin xyz="0 0 0" rpy="0 0 0"/>
+        <geometry>
+            <box size="0.01 0.01 0.01"/>
+        </geometry>
+        </visual>
+        <inertial>
+        <mass value="1e-5" />
+        <origin xyz="0 0 0" rpy="0 0 0"/>
+        <inertia ixx="1e-6" ixy="0" ixz="0" iyy="1e-6" iyz="0" izz="1e-6" />
+        </inertial>
+    </link>
+    <gazebo reference="base_sonar_front_left">
+    <sensor type="ray" name="TeraRanger">
+        <pose>0 0 0 0 0 0</pose>
+        <visualize>true</visualize>
+        <update_rate>50</update_rate>
+        <ray>
+            <scan>
+                <horizontal>
+                <samples>10</samples>
+                <resolution>1</resolution>
+                <min_angle>-0.14835</min_angle>
+                <max_angle>0.14835</max_angle>
+                </horizontal>
+                <vertical>
+                <samples>10</samples>
+                <resolution>1</resolution>
+                <min_angle>-0.14835</min_angle>
+                <max_angle>0.14835</max_angle>
+                </vertical>
+            </scan>
+            <range>
+                <min>0.01</min>
+                <max>2</max>
+                <resolution>0.02</resolution>
+            </range>
+        </ray>
+        <plugin filename="libgazebo_ros_range.so" name="gazebo_ros_range">
+            <gaussianNoise>0.005</gaussianNoise>
+            <alwaysOn>true</alwaysOn>
+            <updateRate>50</updateRate>
+            <topicName>sensor/sonar_front_left</topicName>
+            <frameName>base_sonar_front_left</frameName>
+            <fov>0.2967</fov>
+        </plugin>
+    </sensor>
+    </gazebo>
+    <!-- SONAR SENSOR LEFT-->
+    <joint name="sonar_left_joint" type="fixed">
+    <axis xyz="0 1 0" />
+    <origin rpy="0 0 ${pi/2}" xyz="0.2765 0.112925 0.10134" />
+    <parent link="base_link"/>
+    <child link="base_sonar_left"/>
+    </joint>
+    <link name="base_sonar_left">
+        <collision>
+        <origin xyz="0 0 0" rpy="0 0 0"/>
+        <geometry>
+            <box size="0.01 0.01 0.01"/>
+        </geometry>
+        </collision>
+        <visual>
+        <origin xyz="0 0 0" rpy="0 0 0"/>
+        <geometry>
+            <box size="0.01 0.01 0.01"/>
+        </geometry>
+        </visual>
+        <inertial>
+        <mass value="1e-5" />
+        <origin xyz="0 0 0" rpy="0 0 0"/>
+        <inertia ixx="1e-6" ixy="0" ixz="0" iyy="1e-6" iyz="0" izz="1e-6" />
+        </inertial>
+    </link>
+    <gazebo reference="base_sonar_left">
+    <sensor type="ray" name="TeraRanger">
+        <pose>0 0 0 0 0 0</pose>
+        <visualize>true</visualize>
+        <update_rate>50</update_rate>
+        <ray>
+            <scan>
+                <horizontal>
+                <samples>10</samples>
+                <resolution>1</resolution>
+                <min_angle>-0.14835</min_angle>
+                <max_angle>0.14835</max_angle>
+                </horizontal>
+                <vertical>
+                <samples>10</samples>
+                <resolution>1</resolution>
+                <min_angle>-0.14835</min_angle>
+                <max_angle>0.14835</max_angle>
+                </vertical>
+            </scan>
+            <range>
+                <min>0.01</min>
+                <max>2</max>
+                <resolution>0.02</resolution>
+            </range>
+        </ray>
+        <plugin filename="libgazebo_ros_range.so" name="gazebo_ros_range">
+            <gaussianNoise>0.005</gaussianNoise>
+            <alwaysOn>true</alwaysOn>
+            <updateRate>50</updateRate>
+            <topicName>sensor/sonar_left</topicName>
+            <frameName>base_sonar_left</frameName>
+            <fov>0.2967</fov>
+        </plugin>
+    </sensor>
+    </gazebo>
+    <!-- SONAR SENSOR RIGHT-->
+    <joint name="sonar_right_joint" type="fixed">
+    <axis xyz="0 1 0" />
+    <origin rpy="0 0 -${pi/2}" xyz="0.2765 -0.112925 0.10134" />
+    <parent link="base_link"/>
+    <child link="base_sonar_right"/>
+    </joint>
+    <link name="base_sonar_right">
+        <collision>
+        <origin xyz="0 0 0" rpy="0 0 0"/>
+        <geometry>
+            <box size="0.01 0.01 0.01"/>
+        </geometry>
+        </collision>
+        <visual>
+        <origin xyz="0 0 0" rpy="0 0 0"/>
+        <geometry>
+            <box size="0.01 0.01 0.01"/>
+        </geometry>
+        </visual>
+        <inertial>
+        <mass value="1e-5" />
+        <origin xyz="0 0 0" rpy="0 0 0"/>
+        <inertia ixx="1e-6" ixy="0" ixz="0" iyy="1e-6" iyz="0" izz="1e-6" />
+        </inertial>
+    </link>
+    <gazebo reference="base_sonar_right">
+    <sensor type="ray" name="TeraRanger">
+        <pose>0 0 0 0 0 0</pose>
+        <visualize>true</visualize>
+        <update_rate>50</update_rate>
+        <ray>
+            <scan>
+                <horizontal>
+                <samples>10</samples>
+                <resolution>1</resolution>
+                <min_angle>-0.14835</min_angle>
+                <max_angle>0.14835</max_angle>
+                </horizontal>
+                <vertical>
+                <samples>10</samples>
+                <resolution>1</resolution>
+                <min_angle>-0.14835</min_angle>
+                <max_angle>0.14835</max_angle>
+                </vertical>
+            </scan>
+            <range>
+                <min>0.01</min>
+                <max>2</max>
+                <resolution>0.02</resolution>
+            </range>
+        </ray>
+        <plugin filename="libgazebo_ros_range.so" name="gazebo_ros_range">
+            <gaussianNoise>0.005</gaussianNoise>
+            <alwaysOn>true</alwaysOn>
+            <updateRate>50</updateRate>
+            <topicName>sensor/sonar_right</topicName>
+            <frameName>base_sonar_right</frameName>
+            <fov>0.2967</fov>
+        </plugin>
+    </sensor>
+    </gazebo>
 </robot>

Commit message: added raspberry pi and meshes as well as robot description launch file

File: ros2_automower_description/description/robot_core.xacro (robot description, xacro)
@@ -42,8 +42,8 @@
     </link>
     <!-- LEFT WHEEL LINK -->
-    <joint name="left_wheel_joint" type="continuous">
+    <joint name="left_wheel_joint" type="fixed">
         <parent link="base_link"/>
         <child link="left_wheel"/>
-        <origin xyz="0 0.137925 0" rpy="-${pi/2} 0 0" />
+        <origin xyz="0 0.137925 0" rpy="-1.571 0 0" />
         <axis xyz="0 0 1"/>
     </joint>
@@ -68,5 +68,5 @@
         <parent link="base_link"/>
         <child link="right_wheel"/>
-        <origin xyz="0 -0.137925 " rpy="${pi/2} 0 0" />
+        <origin xyz="0 -0.137925 0" rpy="${pi/2} 0 0" />
         <axis xyz="0 0 -1"/>
     </joint>
@@ -108,4 +108,17 @@
             <origin xyz="0 0 0" rpy="0 0 0"/>
         </xacro:inertial_sphere>
+    </link>
+    <joint name="raspberry_pi_joint" type="fixed">
+        <parent link="chassis"/>
+        <child link="raspberry_pi"/>
+        <origin xyz="0.29215 -0.0109 0.015"/>
+    </joint>
+    <link name="raspberry_pi">
+        <visual>
+            <geometry>
+                <mesh filename="package://ros2_automower_description/meshes/pi_3b.stl"/>
+            </geometry>
+            <material name="blue"/>
+        </visual>
     </link>
     <!-- SENSORS -->
@@ -174,26 +187,26 @@
     <!-- SONAR SENSOR FRONT RIGHT -->
     <joint name="sonar_front_left_joint" type="fixed">
-    <axis xyz="0 1 0" />
-    <origin rpy="0 0 0" xyz="0.41966 0.039825 0.10134" />
-    <parent link="base_link"/>
-    <child link="base_sonar_front_left"/>
+        <axis xyz="0 1 0" />
+        <origin rpy="0 0 0" xyz="0.41966 0.039825 0.10134" />
+        <parent link="base_link"/>
+        <child link="base_sonar_front_left"/>
     </joint>
     <link name="base_sonar_front_left">
         <collision>
-        <origin xyz="0 0 0" rpy="0 0 0"/>
-        <geometry>
-            <box size="0.01 0.01 0.01"/>
-        </geometry>
-        </collision>
-        <visual>
-        <origin xyz="0 0 0" rpy="0 0 0"/>
-        <geometry>
-            <box size="0.01 0.01 0.01"/>
-        </geometry>
+            <origin xyz="0 0 0" rpy="0 0 0"/>
+            <geometry>
+                <box size="0.01 0.01 0.01"/>
+            </geometry>
+        </collision>
+        <visual>
+            <origin xyz="0 0 0" rpy="0 0 0"/>
+            <geometry>
+                <box size="0.01 0.01 0.01"/>
+            </geometry>
         </visual>
         <inertial>
-        <mass value="1e-5" />
-        <origin xyz="0 0 0" rpy="0 0 0"/>
-        <inertia ixx="1e-6" ixy="0" ixz="0" iyy="1e-6" iyz="0" izz="1e-6" />
+            <mass value="1e-5" />
+            <origin xyz="0 0 0" rpy="0 0 0"/>
+            <inertia ixx="1e-6" ixy="0" ixz="0" iyy="1e-6" iyz="0" izz="1e-6" />
         </inertial>
     </link>

Commit message: added kinect

File: ros2_automower_description/description/robot_core.xacro (robot description, xacro)
@@ -42,8 +42,8 @@
     </link>
     <!-- LEFT WHEEL LINK -->
-    <joint name="left_wheel_joint" type="fixed">
+    <joint name="left_wheel_joint" type="continuous">
         <parent link="base_link"/>
         <child link="left_wheel"/>
-        <origin xyz="0 0.137925 0" rpy="-1.571 0 0" />
+        <origin xyz="0 0.137925 0" rpy="-${pi/2} 0 0" />
         <axis xyz="0 0 1"/>
     </joint>
@@ -112,5 +112,5 @@
         <parent link="chassis"/>
         <child link="raspberry_pi"/>
-        <origin xyz="0.29215 -0.0109 0.015"/>
+        <origin xyz="0.29215 -0.04559 0.015"/>
     </joint>
     <link name="raspberry_pi">
@@ -123,4 +123,60 @@
     </link>
     <!-- SENSORS -->
+    <!-- CAMERA -->
+    <joint name="camera_joint" type="fixed">
+        <axis xyz="0 1 0" />
+        <origin rpy="0 0 0" xyz="0.52547 0 0.25614" />
+        <parent link="chassis"/>
+        <child link="camera"/>
+    </joint>
+    <link name="camera">
+        <visual>
+            <geometry>
+                <mesh filename="package://ros2_automower_description/meshes/Kinect.stl"/>
+            </geometry>
+            <material name="blue"/>
+        </visual>
+    </link>
+    <gazebo reference="camera">
+    <sensor name="camera" type="depth">
+        <update_rate>20</update_rate>
+        <camera>
+        <horizontal_fov>1.047198</horizontal_fov>
+        <image>
+            <width>640</width>
+            <height>480</height>
+            <format>R8G8B8</format>
+        </image>
+        <clip>
+            <near>0.05</near>
+            <far>3</far>
+        </clip>
+        </camera>
+        <plugin name="camera_controller" filename="libgazebo_ros_openni_kinect.so">
+        <baseline>0.2</baseline>
+        <alwaysOn>true</alwaysOn>
+        <updateRate>1.0</updateRate>
+        <cameraName>camera_ir</cameraName>
+        <imageTopicName>/camera/color/image_raw</imageTopicName>
+        <cameraInfoTopicName>/camera/color/camera_info</cameraInfoTopicName>
+        <depthImageTopicName>/camera/depth/image_raw</depthImageTopicName>
+        <depthImageInfoTopicName>/camera/depth/camera_info</depthImageInfoTopicName>
+        <pointCloudTopicName>/camera/depth/points</pointCloudTopicName>
+        <frameName>camera</frameName>
+        <pointCloudCutoff>0.5</pointCloudCutoff>
+        <pointCloudCutoffMax>3.0</pointCloudCutoffMax>
+        <distortionK1>0.00000001</distortionK1>
+        <distortionK2>0.00000001</distortionK2>
+        <distortionK3>0.00000001</distortionK3>
+        <distortionT1>0.00000001</distortionT1>
+        <distortionT2>0.00000001</distortionT2>
+        <CxPrime>0</CxPrime>
+        <Cx>0</Cx>
+        <Cy>0</Cy>
+        <focalLength>0</focalLength>
+        <hackBaseline>0</hackBaseline>
+        </plugin>
+    </sensor>
+    </gazebo>
     <!-- SONAR SENSOR FRONT RIGHT -->
     <joint name="sonar_front_right_joint" type="fixed">
