Commit message: added power contacts:

File: ros2_automower_description/description/robot_core.xacro (robot description, xacro)
@@ -37,7 +37,7 @@
             </geometry>
         </collision>
-        <xacro:inertial_box mass="0.5" x="0.57523" y="0.22585" z="0.22935">
+        <!-- <xacro:inertial_box mass="0.5" x="0.57523" y="0.22585" z="0.22935">
             <origin xyz="0.287615 0 0.114675" rpy="0 0 0"/>
-        </xacro:inertial_box>
+        </xacro:inertial_box> -->
     </link>
     <!-- LEFT WHEEL LINK -->
@@ -109,4 +109,5 @@
         </xacro:inertial_sphere>
     </link>
+    <!-- RASPBERRY PI -->
     <joint name="raspberry_pi_joint" type="fixed">
         <parent link="chassis"/>
@@ -122,5 +123,139 @@
         </visual>
     </link>
+    <!-- CHARGING CONTACTS -->
+    <joint name="left_charging_contact_joint" type="fixed">
+        <parent link="chassis"/>
+        <child link="left_charging_contact_link"/>
+        <origin xyz="-0.02535 0.06 0.11647"/>
+    </joint>
+    <link name="left_charging_contact_link">
+        <visual>
+            <geometry>
+                <mesh filename="package://ros2_automower_description/meshes/left_power_contact.stl"/>
+            </geometry>
+            <material name="blue"/>
+        </visual>
+        <collision>
+            <geometry>
+                <mesh filename="package://ros2_automower_description/meshes/left_power_contact.stl"/>
+            </geometry>
+        </collision>
+    </link>
+    <joint name="right_charging_contact_joint" type="fixed">
+        <parent link="chassis"/>
+        <child link="right_charging_contact_link"/>
+        <origin xyz="-0.02535 -0.06 0.11647"/>
+    </joint>
+    <link name="right_charging_contact_link">
+        <visual>
+            <geometry>
+                <mesh filename="package://ros2_automower_description/meshes/right_power_contact.stl"/>
+            </geometry>
+            <material name="blue"/>
+        </visual>
+        <collision>
+            <geometry>
+                <mesh filename="package://ros2_automower_description/meshes/right_power_contact.stl"/>
+            </geometry>
+        </collision>
+    </link>
     <!-- SENSORS -->
+    <!-- GPS -->
+    <joint name="gps_joint" type="fixed">
+        <parent link="chassis"/>
+        <child link="gps_link"/>
+        <origin xyz="0.34488 0 0.23987" />
+    </joint>
+    <link name="gps_link">
+        <visual>
+            <geometry>
+                <box size="0.04 0.04 0.04"/>
+            </geometry>
+            <material name="blue"/>
+        </visual>
+    </link>
+    <gazebo reference="gps_link">
+        <sensor name="gps_sensor" type="gps">
+            <always_on>true</always_on>
+            <update_rate>1.0</update_rate>
+            <plugin name="gps_controller" filename="libgazebo_ros_gps_sensor.so">
+                <ros>
+                    <!-- <namespace>/br</namespace> -->
+                    <remapping>gps_controller/out:=gps</remapping>
+                </ros>
+                <frame_name>gps_link</frame_name>
+            </plugin>
+        </sensor>
+        <material>Gazebo/Grey</material>
+    </gazebo>
+    <!--IMU-->
+    <joint name="imu_joint" type="fixed">
+        <parent link="raspberry_pi"/>
+        <child link="imu_link"/>
+        <origin xyz="-0.02756 0.06226 0" rpy="0 0 ${pi}"/>
+    </joint>
+    <link name="imu_link">
+        <visual>
+            <geometry>
+                <mesh filename="package://ros2_automower_description/meshes/GY-521_imu.stl" scale="0.1 0.1 0.1"/>
+            </geometry>
+            <material name="blue"/>
+        </visual>
+    </link>
+    <gazebo reference="imu_link">
+        <sensor name="br_imu" type="imu">
+            <always_on>true</always_on>
+            <update_rate>100</update_rate>
+            <imu>
+            <angular_velocity>
+                <x>
+                <noise type="gaussian">
+                    <mean>0.0</mean>
+                    <stddev>2e-4</stddev>
+                </noise>
+                </x>
+                <y>
+                <noise type="gaussian">
+                    <mean>0.0</mean>
+                    <stddev>2e-4</stddev>
+                </noise>
+                </y>
+                <z>
+                <noise type="gaussian">
+                    <mean>0.0</mean>
+                    <stddev>2e-4</stddev>
+                </noise>
+                </z>
+            </angular_velocity>
+            <linear_acceleration>
+                <x>
+                <noise type="gaussian">
+                    <mean>0.0</mean>
+                    <stddev>1.7e-2</stddev>
+                </noise>
+                </x>
+                <y>
+                <noise type="gaussian">
+                    <mean>0.0</mean>
+                    <stddev>1.7e-2</stddev>
+                </noise>
+                </y>
+                <z>
+                <noise type="gaussian">
+                    <mean>0.0</mean>
+                    <stddev>1.7e-2</stddev>
+                </noise>
+                </z>
+            </linear_acceleration>
+            </imu>
+            <plugin name="bytes_imu" filename="libgazebo_ros_imu_sensor.so">
+                <ros>
+                    <namespace>imu</namespace>
+                    <remapping>~/out:=data</remapping>
+                </ros>
+                <initial_orientation_as_reference>false</initial_orientation_as_reference>
+            </plugin>
+        </sensor>
+    </gazebo>
     <!-- CAMERA -->
     <joint name="camera_joint" type="fixed">
@@ -139,50 +274,50 @@
     </link>
     <gazebo reference="camera">
-    <sensor name="camera" type="depth">
-        <update_rate>20</update_rate>
-        <camera>
-        <horizontal_fov>1.047198</horizontal_fov>
-        <image>
-            <width>640</width>
-            <height>480</height>
-            <format>R8G8B8</format>
-        </image>
-        <clip>
-            <near>0.05</near>
-            <far>3</far>
-        </clip>
-        </camera>
-        <plugin name="camera_controller" filename="libgazebo_ros_openni_kinect.so">
-        <baseline>0.2</baseline>
-        <alwaysOn>true</alwaysOn>
-        <updateRate>1.0</updateRate>
-        <cameraName>camera_ir</cameraName>
-        <imageTopicName>/camera/color/image_raw</imageTopicName>
-        <cameraInfoTopicName>/camera/color/camera_info</cameraInfoTopicName>
-        <depthImageTopicName>/camera/depth/image_raw</depthImageTopicName>
-        <depthImageInfoTopicName>/camera/depth/camera_info</depthImageInfoTopicName>
-        <pointCloudTopicName>/camera/depth/points</pointCloudTopicName>
-        <frameName>camera</frameName>
-        <pointCloudCutoff>0.5</pointCloudCutoff>
-        <pointCloudCutoffMax>3.0</pointCloudCutoffMax>
-        <distortionK1>0.00000001</distortionK1>
-        <distortionK2>0.00000001</distortionK2>
-        <distortionK3>0.00000001</distortionK3>
-        <distortionT1>0.00000001</distortionT1>
-        <distortionT2>0.00000001</distortionT2>
-        <CxPrime>0</CxPrime>
-        <Cx>0</Cx>
-        <Cy>0</Cy>
-        <focalLength>0</focalLength>
-        <hackBaseline>0</hackBaseline>
-        </plugin>
-    </sensor>
+        <sensor name="camera" type="depth">
+            <update_rate>20</update_rate>
+            <camera>
+            <horizontal_fov>1.047198</horizontal_fov>
+            <image>
+                <width>640</width>
+                <height>480</height>
+                <format>R8G8B8</format>
+            </image>
+            <clip>
+                <near>0.05</near>
+                <far>3</far>
+            </clip>
+            </camera>
+            <plugin name="camera_controller" filename="libgazebo_ros_openni_kinect.so">
+            <baseline>0.2</baseline>
+            <alwaysOn>true</alwaysOn>
+            <updateRate>1.0</updateRate>
+            <cameraName>camera_ir</cameraName>
+            <imageTopicName>/camera/color/image_raw</imageTopicName>
+            <cameraInfoTopicName>/camera/color/camera_info</cameraInfoTopicName>
+            <depthImageTopicName>/camera/depth/image_raw</depthImageTopicName>
+            <depthImageInfoTopicName>/camera/depth/camera_info</depthImageInfoTopicName>
+            <pointCloudTopicName>/camera/depth/points</pointCloudTopicName>
+            <frameName>camera</frameName>
+            <pointCloudCutoff>0.5</pointCloudCutoff>
+            <pointCloudCutoffMax>3.0</pointCloudCutoffMax>
+            <distortionK1>0.00000001</distortionK1>
+            <distortionK2>0.00000001</distortionK2>
+            <distortionK3>0.00000001</distortionK3>
+            <distortionT1>0.00000001</distortionT1>
+            <distortionT2>0.00000001</distortionT2>
+            <CxPrime>0</CxPrime>
+            <Cx>0</Cx>
+            <Cy>0</Cy>
+            <focalLength>0</focalLength>
+            <hackBaseline>0</hackBaseline>
+            </plugin>
+        </sensor>
     </gazebo>
     <!-- SONAR SENSOR FRONT RIGHT -->
     <joint name="sonar_front_right_joint" type="fixed">
-    <axis xyz="0 1 0" />
-    <origin rpy="0 0 0" xyz="0.41966 -0.039825 0.10134" />
-    <parent link="base_link"/>
-    <child link="base_sonar_front_right"/>
+        <axis xyz="0 1 0" />
+        <origin rpy="0 0 0" xyz="0.41966 -0.039825 0.10134" />
+        <parent link="base_link"/>
+        <child link="base_sonar_front_right"/>
     </joint>
     <link name="base_sonar_front_right">

Commit message: add sim control

File: ros2_automower_description/description/robot_core.xacro (robot description, xacro)
@@ -41,4 +41,7 @@
         </xacro:inertial_box> -->
     </link>
+    <gazebo reference="chassis">
+        <material>Gazebo/white</material>
+    </gazebo>
     <!-- LEFT WHEEL LINK -->
     <joint name="left_wheel_joint" type="continuous">
@@ -64,4 +67,7 @@
         </xacro:inertial_cylinder>
     </link>
+    <gazebo reference="left_wheel">
+        <material>Gazebo/blue</material>
+    </gazebo>
     <!-- RIGHT WHEEL LINK -->
     <joint name="right_wheel_joint" type="continuous">
@@ -87,4 +93,7 @@
         </xacro:inertial_cylinder>
     </link>
+    <gazebo reference="right_wheel">
+        <material>Gazebo/blue</material>
+    </gazebo>
     <!-- CASTER WHEEL LINK -->
     <joint name="caster_wheel_joint" type="fixed">
@@ -109,4 +118,9 @@
         </xacro:inertial_sphere>
     </link>
+    <gazebo reference="caster_wheel">
+        <material>Gazebo/black</material>
+        <mu1 value="0.0001"/>
+        <mu2 value="0.0001"/>
+    </gazebo>
     <!-- RASPBERRY PI -->
     <joint name="raspberry_pi_joint" type="fixed">

Commit message: move caster down

File: ros2_automower_description/description/robot_core.xacro (robot description, xacro)
@@ -100,5 +100,5 @@
         <parent link="chassis"/>
         <child link="caster_wheel"/>
-        <origin xyz="0.41 0 0"/>
+        <origin xyz="0.41 0 -0.1"/>
     </joint>
     <link name="caster_wheel">

Commit message: move caster

File: ros2_automower_description/description/robot_core.xacro (robot description, xacro)
@@ -100,5 +100,5 @@
         <parent link="chassis"/>
         <child link="caster_wheel"/>
-        <origin xyz="0.41 0 -0.1"/>
+        <origin xyz="0.41 0 -0.0.025"/>
     </joint>
     <link name="caster_wheel">

Commit message: added multicamera

File: ros2_automower_description/description/robot_core.xacro (robot description, xacro)
@@ -100,5 +100,5 @@
         <parent link="chassis"/>
         <child link="caster_wheel"/>
-        <origin xyz="0.41 0 -0.1"/>
+        <origin xyz="0.41 0 -0.025"/>
     </joint>
     <link name="caster_wheel">
@@ -287,5 +287,5 @@
         </visual>
     </link>
-    <gazebo reference="camera">
+    <!-- <gazebo reference="camera">
         <sensor name="camera" type="depth">
             <update_rate>20</update_rate>
@@ -327,4 +327,59 @@
             </plugin>
         </sensor>
+    </gazebo> -->
+    <gazebo reference="camera">
+        <sensor type="multicamera" name="stereo_camera">
+        <update_rate>30.0</update_rate>
+        <camera name="left">
+            <horizontal_fov>1.3962634</horizontal_fov>
+            <image>
+            <width>800</width>
+            <height>800</height>
+            <format>R8G8B8</format>
+            </image>
+            <clip>
+            <near>0.02</near>
+            <far>300</far>
+            </clip>
+            <noise>
+            <type>gaussian</type>
+            <mean>0.0</mean>
+            <stddev>0.007</stddev>
+            </noise>
+        </camera>
+        <camera name="right">
+            <pose>0 -0.07 0 0 0 0</pose>
+            <horizontal_fov>1.3962634</horizontal_fov>
+            <image>
+            <width>800</width>
+            <height>800</height>
+            <format>R8G8B8</format>
+            </image>
+            <clip>
+            <near>0.02</near>
+            <far>300</far>
+            </clip>
+            <noise>
+            <type>gaussian</type>
+            <mean>0.0</mean>
+            <stddev>0.007</stddev>
+            </noise>
+        </camera>
+        <plugin name="stereo_camera_controller" filename="libgazebo_ros_camera.so">
+            <alwaysOn>true</alwaysOn>
+            <updateRate>0.0</updateRate>
+            <cameraName>multisense_sl/camera</cameraName>
+            <imageTopicName>image_raw</imageTopicName>
+            <cameraInfoTopicName>camera_info</cameraInfoTopicName>
+            <frameName>left_camera_optical_frame</frameName>
+            <!--<rightFrameName>right_camera_optical_frame</rightFrameName>-->
+            <hackBaseline>0.07</hackBaseline>
+            <distortionK1>0.0</distortionK1>
+            <distortionK2>0.0</distortionK2>
+            <distortionK3>0.0</distortionK3>
+            <distortionT1>0.0</distortionT1>
+            <distortionT2>0.0</distortionT2>
+        </plugin>
+        </sensor>
     </gazebo>
     <!-- SONAR SENSOR FRONT RIGHT -->

Commit message: correct camera frame name

File: ros2_automower_description/description/robot_core.xacro (robot description, xacro)
@@ -277,7 +277,7 @@
         <origin rpy="0 0 0" xyz="0.52547 0 0.25614" />
         <parent link="chassis"/>
-        <child link="camera"/>
-    </joint>
-    <link name="camera">
+        <child link="camera_link"/>
+    </joint>
+    <link name="camera_link">
         <visual>
             <geometry>
@@ -287,5 +287,11 @@
         </visual>
     </link>
-    <gazebo reference="camera">
+    <joint name="camera_optical_joint" type="fixed">
+        <parent link="camera_link"/>
+        <child link="camera_link_optical"/>
+        <origin xyz="0 0 0" rpy="${-pi/2} 0 ${-pi/2}"/>
+    </joint>
+    <link name="camera_link_optical"></link>
+    <gazebo reference="camera_link">
         <sensor name="camera" type="depth">
             <update_rate>20</update_rate>
@@ -312,5 +318,5 @@
             <depthImageInfoTopicName>/camera/depth/camera_info</depthImageInfoTopicName>
             <pointCloudTopicName>/camera/depth/points</pointCloudTopicName>
-            <frameName>camera</frameName>
+            <frameName>camera_link_optical</frameName>
             <pointCloudCutoff>0.5</pointCloudCutoff>
             <pointCloudCutoffMax>3.0</pointCloudCutoffMax>

Commit message: update sim

File: ros2_automower_description/description/robot_core.xacro (robot description, xacro)
@@ -37,7 +37,7 @@
             </geometry>
         </collision>
-        <!-- <xacro:inertial_box mass="0.5" x="0.57523" y="0.22585" z="0.22935">
+        <xacro:inertial_box mass="0.5" x="0.57523" y="0.22585" z="0.22935">
             <origin xyz="0.287615 0 0.114675" rpy="0 0 0"/>
-        </xacro:inertial_box> -->
+        </xacro:inertial_box>
     </link>
     <gazebo reference="chassis">
@@ -293,5 +293,5 @@
     </joint>
     <link name="camera_link_optical"></link>
-    <gazebo reference="camera_link">
+    <!-- <gazebo reference="camera_link">
         <sensor name="camera" type="depth">
             <update_rate>20</update_rate>
@@ -333,6 +333,31 @@
             </plugin>
         </sensor>
-    </gazebo>
-    <!-- <gazebo reference="camera">
+    </gazebo> -->
+    <gazebo reference="camera_link">
+        <material>Gazebo/Red</material>
+    <sensor name="camera" type="depth">
+            <pose> 0 0 0 0 0 0 </pose>
+            <visualize>true</visualize>
+            <update_rate>10</update_rate>
+            <camera>
+                <horizontal_fov>1.089</horizontal_fov>
+                <image>
+                    <format>B8G8R8</format>
+                    <width>640</width>
+                    <height>480</height>
+                </image>
+                <clip>
+                    <near>0.05</near>
+                    <far>8.0</far>
+                </clip>
+            </camera>
+            <plugin name="camera_controller" filename="libgazebo_ros_camera.so">
+                <frame_name>camera_link_optical</frame_name>
+                <min_depth>0.1</min_depth>
+                <max_depth>10.0</max_depth>
+            </plugin>
+        </sensor>
+    </gazebo>
+    <!-- <gazebo reference="camera_link">
         <sensor type="multicamera" name="stereo_camera">
         <update_rate>30.0</update_rate>
@@ -378,6 +403,5 @@
             <imageTopicName>image_raw</imageTopicName>
             <cameraInfoTopicName>camera_info</cameraInfoTopicName>
-            <frameName>left_camera_optical_frame</frameName>
-               ///<rightFrameName>right_camera_optical_frame</rightFrameName>
+            <frameName>amera_optical_frame</frameName>
             <hackBaseline>0.07</hackBaseline>
             <distortionK1>0.0</distortionK1>
